Commit message: Finished 2/3 of module 6

File: ros2_ws/src/toktok_description/urdf/mobile_base.xacro (robot description, xacro)
@@ -12,7 +12,14 @@
                 <box size="${base_length} ${base_width} ${base_height}" />
             </geometry>
-            <origin xyz="0 0 0.1" rpy="0 0 0" />
+            <origin xyz="0 0 ${base_height / 2.0}" rpy="0 0 0" />
             <material name="blue" />
         </visual>
+        <collision>
+            <geometry>
+                <box size="${base_length} ${base_width} ${base_height}" />
+            </geometry>
+            <origin xyz="0 0 ${base_height / 2.0}" rpy="0 0 0" />
+        </collision>
+        <xacro:box_inertial m="5.0" x="${base_length}" y="${base_width}" z="${base_height}" o_xyz = "0 0 ${base_height / 2.0}"  o_rpy ="0 0 0 " />
     </link>
     <xacro:macro name="wheel_link" params="prefix">
@@ -25,4 +32,11 @@
                 <material name="red" />
             </visual>
+            <collision>
+                <geometry>
+                    <sphere radius="${wheel_radius}" />
+                </geometry>
+                <origin xyz="0 0 0" rpy="${pi / 2.0} 0 0" />
+            </collision>
+            <xacro:cylinder_inertial m="1.0" r="${wheel_radius}" l="${wheel_length}" o_xyz="0 0 0" o_rpy="${pi / 2.0} 0 0" />
     </link>
     </xacro:macro>
@@ -37,4 +51,11 @@
             <material name="red" />
         </visual>
+        <collision>
+            <geometry>
+                <sphere radius="${wheel_radius / 2.0}" />
+            </geometry>
+            <origin xyz="0 0 0" rpy="0 0 0" />
+        </collision>
+        <xacro:sphere_inertial m="0.5" r="${wheel_radius / 2.0}" o_xyz = "0 0 0" o_rpy="0 0 0" />
     </link>
     <joint name="base_base" type="fixed">

File: ros2_ws/src/toktok_description/urdf/properties.xacro (robot description, xacro)
@@ -7,3 +7,24 @@
         <color rgba="0 0 0.5 1" />
     </material>
+    <xacro:macro name="box_inertial" params="m x y z o_xyz o_rpy">
+        <inertial>
+            <origin xyz="${o_xyz}" rpy="${o_rpy}" />
+            <mass value="${m}"/>
+            <inertia ixx="${(m/12) * (y*y + z*z)}" ixy="0" ixz="0" iyy="${(m/12) * (x*x + z*z)}" iyz="0" izz="${(m/12) * (y*y + x*x)}"/>
+        </inertial>
+    </xacro:macro>
+    <xacro:macro name="cylinder_inertial" params="m r l o_xyz o_rpy">
+        <inertial>
+            <origin xyz="${o_xyz}" rpy="${o_rpy}" />
+            <mass value="${m}"/>
+            <inertia ixx="${(m/12) * (3*r*r + l*l)}" ixy="0" ixz="0" iyy="${(m/12) * (3*r*r + l*l)}" iyz="0" izz="${(m/2) * (r*r)}"/>
+        </inertial>
+    </xacro:macro>
+    <xacro:macro name="sphere_inertial" params="m r o_xyz o_rpy">
+        <inertial>
+            <origin xyz="${o_xyz}" rpy="${o_rpy}" />
+            <mass value="${m}"/>
+            <inertia ixx="${((2*m/5)*r*r)}" ixy="0" ixz="0" iyy="${((2*m/5)*r*r)}" iyz="0" izz="${((2*m/5)*r*r)}"/>
+        </inertial>
+    </xacro:macro>
 </robot>
